File: 1284-breakout/rev_1.0/rev_1.0.sch (KiCad schematic (older format))
At the start: 18 parts, among them J0 ICSP, SW0 RESET, U0 ATmega1284P-PU, U1 LM1117-5.0, U3 FT232RL, Y0 16MHz

Commit message: added sensor logic subsheets
Parts:
- removed C2: 4.7uF_16V, symbol Device:CP
- removed RP2 (x2): 1k, symbol Device:R
- removed U0: ATmega1284P-PU, Package_DIP:DIP-40_W15.24mm, symbol MCU_Microchip_ATmega:ATmega1284P-PU
- removed U3: FT232RL, Package_SO:SSOP-28_5.3x10.2mm_P0.65mm, symbol Interface_USB:FT232RL
- added BT?: 3V Coin Cell, symbol Device:Battery_Cell
- added C10, C7, C? (x3): 1uF, symbol Device:C
- added C11, C12: 18pF, symbol Device:C_Small
- added C?: 4.7uF_16V, symbol Device:C
- added J1: Micro_SD_Card_Det_Hirose_DM3AT, symbol Connector:Micro_SD_Card_Det_Hirose_DM3AT
- added PLED_3V3: Green, symbol Device:LED
- added RP2: 1k, symbol Device:R
- added RP3, RP4: 1.6k, symbol Device:R
- added U0: ATmega1284-AU, Package_QFP:TQFP-44_10x10mm_P0.8mm, symbol MCU_Microchip_ATmega:ATmega1284-AU
- added U2: MCP7940N-xSN, symbol Timer:MCP7940N-xSN
- added U2: LM1117-3.3, symbol Regulator_Linear:LM1117-5.0
- added U?: TXB0104D, Package_SO:SOIC-14_3.9x8.7mm_P1.27mm, symbol Logic_LevelTranslator:TXB0104D
- added Y1: 32.768 kHz, symbol Device:Crystal_Small
- RP0: value 1k -> 10k
- renumbered J0 to J1, PLED to PLED_5V
Connections:
- net +5V: now also C10.1, C?.1, C?.2, RP3.1, RP4.1, U0.17 (VCC), U0.27 (AVCC), U0.38 (VCC), U0.5 (VCC), U2.8 (VCC), U?.14 (VCCB)
- net A0: now also U0.37 (PA0)
- net A1: now also U0.36 (PA1)
- net A2: now also U0.35 (PA2)
- net A3: now also U0.34 (PA3)
- net A4: now also U0.33 (PA4)
- net A5: now also U0.32 (PA5)
- net A6: now also U0.31 (PA6)
- net A7: now also U0.30 (PA7)
- net AIN0/: now also U0.42 (PB2)
- net AIN1/: now also U0.43 (PB3), U?.10 (B4)
- net CLKO/: now also U0.41 (PB1)
- net GND: now also BT?.2 (-), C10.2, C11.2, C12.1, C7.2, C?.1, C?.2, C?.2, C?.2, J1.6 (VSS), PLED_3V3.1 (K), U0.18 (GND), U0.28 (GND), U0.39 (GND), U0.6 (GND), U2.1 (GND), U2.4 (VSS)
- net ICP1/: now also U0.15 (PD6)
- net MISO: now also U0.2 (PB6), U?.12 (B2)
- net MOSI: now also U0.1 (PB5), U?.13 (B1)
- net OC1A/: now also U0.14 (PD5)
- net OC1B/: now also U0.13 (PD4)
- net OC2A/: now also U0.16 (PD7)
- net PCINT18: now also U0.21 (PC2)
- net PCINT19: now also U0.22 (PC3)
- net PCINT20: now also U0.23 (PC4)
- net PCINT21: now also U0.24 (PC5)
- net PCINT22: now also U0.25 (PC6)
- net PCINT23: now also U0.26 (PC7)
- net PCINT8: now also U0.40 (PB0)
- net RESET: now also RP0.2, SW0.2, U0.4 (~RESET)
- net RX0: now also U0.9 (PD0)
- net RX1: now also U0.11 (PD2)
- net SCK: now also U0.3 (PB7), U?.11 (B3)
- net SCL: now also RP4.2, U0.19 (PC0), U2.6 (SCL)
- net SDA: now also RP3.2, U0.20 (PC1), U2.5 (SDA)
- net SS: now also U0.44 (PB4)
- net TX0: now also U0.10 (PD1)
- net TX1: now also U0.12 (PD3)
- net Vsupply: now also U2.3 (VI)
- net XTAL1: now also U0.8 (XTAL1)
- net XTAL2: now also U0.7 (XTAL2)
- net at C0.2: now also U0.29 (AREF)
- new net: C12.2, U2.1 (X1), Y1.1
- new net: C11.1, U2.2 (X2), Y1.2
- new net: BT?.1 (+), U2.3 (VBAT)
- new net: PLED_3V3.2 (A), RP2.1
- new net +3V3: C7.1, C?.1, C?.1, J1.4 (VDD), RP2.2, U2.2 (VO), U?.1 (VCCA), U?.8 (OE)
- new net CS_3V3: J1.2 (DAT3/CD), U?.5 (A4)
- new net MISO_3V3: J1.7 (DAT0), U?.3 (A2)
- new net MOSI_3V3: J1.3 (CMD), U?.2 (A1)
- new net SCK_3V3: J1.5 (CLK), U?.4 (A3)
- no-connect marks 0 -> 6
Other:
- note added: "3V3 Voltage Regulation"
- note added: "I2C Pullup\n"
- note added: "Level Shifter\n"
- note added: "Li-Po Battery\nConnector\n"
- note added: "MicroSD\n"
- note added: "Microcontroller\n[AtMEGA1284P-AU]"
- note added: "RTC Module\n"
- note removed: "Microcontroller\n[AtMEGA1284P-PU]"
- moved on the sheet: C4, C5, RP0, SW0, Y0

Commit message: begin routing
Parts:
- removed RP0: 10k, symbol Device:R
- removed SW0: RESET, symbol Switch:SW_Push
- added C10, C11, C12, C9: 0.1uF, Capacitor_SMD:C_0402_1005Metric, symbol Device:C
- added CAN1: SPI_CAN_BREAKOUT, TestBaja:CAN_Module, symbol Connector:Conn_01x16_Female
- added J10: RR_rh, Connector_PinHeader_2.54mm:PinHeader_1x03_P2.54mm_Vertical, symbol Connector:Conn_01x03_Female
- added J11: Tach, Connector_PinHeader_2.54mm:PinHeader_1x03_P2.54mm_Vertical, symbol Connector:Conn_01x03_Female
- added J12: MAX31865, TestBaja:RTD, symbol Connector:Conn_01x08_Female
- added J14: Ulti_GPS_v3, baja1920:UltiGPSv3, symbol Connector:Conn_01x09_Female
- added J2: RF_BHE, Connector_PinHeader_2.54mm:PinHeader_1x03_P2.54mm_Vertical, symbol Connector:Conn_01x03_Female
- added J3: Output_BHE, Connector_PinHeader_2.54mm:PinHeader_1x03_P2.54mm_Vertical, symbol Connector:Conn_01x03_Female
- added J4: IMU_bout, baja1920:6dof_MPU6050, symbol Connector:Conn_01x05_Female
- added J5: LF_BHE, Connector_PinHeader_2.54mm:PinHeader_1x03_P2.54mm_Vertical, symbol Connector:Conn_01x03_Female
- added J6: CVT_IR, Connector_PinHeader_2.54mm:PinHeader_1x04_P2.54mm_Vertical, symbol Connector:Conn_01x04_Female
- added J7: LF_rh, Connector_PinHeader_2.54mm:PinHeader_1x03_P2.54mm_Vertical, symbol Connector:Conn_01x03_Female
- added J8: LR_rh, Connector_PinHeader_2.54mm:PinHeader_1x03_P2.54mm_Vertical, symbol Connector:Conn_01x03_Female
- added J9: RF_rh, Connector_PinHeader_2.54mm:PinHeader_1x03_P2.54mm_Vertical, symbol Connector:Conn_01x03_Female
- added POWER1: Vsupply, baja1920:Power, symbol Connector:Conn_01x02_Female
- added R1: 1M, Resistor_SMD:R_0402_1005Metric, symbol Device:R
- added R2, R3, R6: 4.7k, Resistor_SMD:R_0402_1005Metric, symbol Device:R_Small
- added R4, R5, R7: 1k, Resistor_SMD:R_0402_1005Metric, symbol Device:R_Small
- added RP1, RP9: 10k, Resistor_SMD:R_0402_1005Metric, symbol Device:R
- added RP5, RP6, RP7: 1k, Resistor_SMD:R_0402_1005Metric, symbol Device:R
- added SW1: BT_RST, Button_Switch_SMD:SW_SPST_EVQQ2, symbol Switch:SW_Push
- added U3, U4: TXB0104D, Package_SO:SOIC-14_3.9x8.7mm_P1.27mm, symbol Logic_LevelTranslator:TXB0104D
- BT1: renamed from BT?; footprint (none) -> Battery:BatteryHolder_Keystone_1058_1x2032; Part URL (none) -> https://www.digikey.com/product-detail/en/keystone-electron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
- C1, C3, C6, C7: footprint (none) -> Capacitor_SMD:C_0603_1608Metric; Part URL (none) -> https://www.digikey.com/product-detail/en/samsung-electro-m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
- C13, C14: renamed from C?; value 1uF -> 0.1uF; footprint (none) -> Capacitor_SMD:C_0402_1005Metric; Part URL (none) -> https://www.digikey.com/product-detail/en/yageo/CC0402KRX7R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
- C15: renamed from C?; footprint (none) -> Capacitor_SMD:C_0603_1608Metric; Part URL (none) -> https://www.digikey.com/product-detail/en/samsung-electro-m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
- C16: renamed from C10; footprint (none) -> Capacitor_SMD:C_0603_1608Metric; Part URL (none) -> https://www.digikey.com/product-detail/en/samsung-electro-m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
- C17: renamed from C12; footprint (none) -> Capacitor_SMD:C_0201_0603Metric; Part URL (none) -> https://www.digikey.com/product-detail/en/murata-electronic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
- C18: renamed from C11; footprint (none) -> Capacitor_SMD:C_0201_0603Metric; Part URL (none) -> https://www.digikey.com/product-detail/en/murata-electronic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
- C2: renamed from C0; value 100nf -> 0.1uF; footprint (none) -> Capacitor_SMD:C_0402_1005Metric; Part URL (none) -> https://www.digikey.com/product-detail/en/yageo/CC0402KRX7R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
- C4, C5: value 22pf -> 20pF; footprint (none) -> Capacitor_SMD:C_0201_0603Metric; Part URL (none) -> https://www.digikey.com/product-detail/en/murata-electronic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
- C8: renamed from C?; footprint (none) -> Capacitor_SMD:C_0805_2012Metric; Part URL (none) -> https://www.digikey.com/product-detail/en/w-rth-elektronik/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
- J1: footprint (none) -> Connector_PinHeader_2.54mm:PinHeader_2x03_P2.54mm_Vertical
- J13: renamed from J1; footprint (none) -> Connector_Card:microSD_HC_Hirose_DM3AT-SF-PEJM5; Part URL (none) -> https://www.digikey.com/product-detail/en/gct/MEM2075-00-14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
- PLED_3V3: footprint (none) -> LED_SMD:LED_0603_1608Metric; Part URL (none) -> https://www.digikey.com/product-detail/en/w-rth-elektronik/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
- PLED_5V1: renamed from PLED_5V; footprint (none) -> LED_SMD:LED_0603_1608Metric; Part URL (none) -> https://www.digikey.com/product-detail/en/w-rth-elektronik/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
- RP2: footprint (none) -> Resistor_SMD:R_0402_1005Metric; Part URL (none) -> https://www.digikey.com/product-detail/en/panasonic-electro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
- RP3: renamed from RP4; value 1.6k -> 4.7k; footprint (none) -> Resistor_SMD:R_0402_1005Metric; Part URL (none) -> https://www.digikey.com/product-detail/en/panasonic-electro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
- RP4: renamed from RP3; value 1.6k -> 4.7k; footprint (none) -> Resistor_SMD:R_0402_1005Metric; Part URL (none) -> https://www.digikey.com/product-detail/en/panasonic-electro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
- RP8: renamed from RP1; footprint (none) -> Resistor_SMD:R_0402_1005Metric; Part URL (none) -> https://www.digikey.com/product-detail/en/panasonic-electro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
- U0: Part URL (none) -> https://www.digikey.com/product-detail/en/microchip-technol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
- U1, U2: footprint (none) -> Package_TO_SOT_SMD:SOT-223; Part URL (none) -> https://www.digikey.com/product-detail/en/texas-instruments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
- U5: renamed from U?; Part URL (none) -> https://www.digikey.com/product-detail/en/texas-instruments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
- U6: renamed from U2; footprint (none) -> Package_SO:SOIC-8_3.9x4.9mm_P1.27mm; Part URL (none) -> https://www.digikey.com/product-detail/en/microchip-technol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
- Y1: renamed from Y0; footprint (none) -> Crystal:Crystal_SMD_HC49-SD; Part URL (none) -> https://www.digikey.com/product-detail/en/ecs-inc/ECS-160-2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
- Y2: renamed from Y1; footprint (none) -> Crystal:Crystal_SMD_3215-2Pin_3.2x1.5mm; Part URL (none) -> https://www.digikey.com/product-detail/en/epson/FC-135-32.7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
Connections:
- net +3V3: now also C10.1, C9.1, RP5.1, RP6.1, RP7.1, U3.1 (VCCA), U4.1 (VCCA); no longer U5.8 (OE)
- net +5V: now also C11.2, C12.2, CAN1.15 (Pin_15), J10.2 (Pin_2), J11.2 (Pin_2), J12.1 (Pin_1), J14.8 (Pin_8), J4.1 (Pin_1), J6.3 (Pin_3), J7.2 (Pin_2), J8.2 (Pin_2), J9.2 (Pin_2), RP1.1, RP9.2, U3.14 (VCCB), U4.14 (VCCB)
- net A0: now also J7.1 (Pin_1)
- net A1: now also J9.1 (Pin_1)
- net A2: now also J8.1 (Pin_1)
- net A3: now also J10.1 (Pin_1)
- net GND: now also J13.11 (SHIELD), U5.7 (GND), C10.2, C11.1, C12.1, C9.2, CAN1.1 (Pin_1), CAN1.16 (Pin_16), J10.3 (Pin_3), J11.3 (Pin_3), J12.2 (Pin_2), J14.7 (Pin_7), J2.2 (Pin_2), J3.2 (Pin_2), J4.2 (Pin_2), J5.2 (Pin_2), J6.4 (Pin_4), J7.3 (Pin_3), J8.3 (Pin_3), J9.3 (Pin_3), POWER1.2 (Pin_2), R2.1, R3.1, R6.1, SW1.1, U3.7 (GND), U4.7 (GND)
- net MISO: now also CAN1.4 (Pin_4), J12.5 (Pin_5)
- net MOSI: now also CAN1.3 (Pin_3), J12.6 (Pin_6)
- net PCINT18: now also U3.11 (B3)
- net PCINT19: now also U3.10 (B4)
- net PCINT20: now also U4.12 (B2)
- net PCINT21: now also U4.11 (B3)
- net PCINT22: now also U4.10 (B4)
- net PCINT23: now also J4.5 (Pin_5)
- net PCINT8: now also J11.1 (Pin_1)
- net RESET: now also CAN1.7 (Pin_7), RP1.2, SW1.2
- net RX0: now also J14.5 (Pin_5)
- net RX1: now also U3.13 (B1)
- net SCK: now also CAN1.5 (Pin_5), J12.4 (Pin_4)
- net SCL: now also J4.4 (Pin_4), J6.2 (Pin_2)
- net SDA: now also J4.3 (Pin_3), J6.1 (Pin_1)
- net TX0: now also J14.6 (Pin_6)
- net TX1: now also U3.12 (B2)
- net XTAL1: now also R1.1
- net XTAL2: now also R1.2
- net AIN0/ renamed PCINT10
- net PCINT10: now also R6.2, R7.2
- net AIN1/ renamed PCINT11
- net PCINT11: now also R3.2, R5.2; no longer U5.10 (B4)
- net CLKO/ renamed PCINT9
- net PCINT9: now also R2.2, R4.2
- net ICP1/ renamed PCINT30
- net PCINT30: now also CAN1.6 (Pin_6)
- net OC1A/ renamed PCINT29
- net PCINT29: now also J12.7 (Pin_7)
- net OC1B/ renamed PCINT28
- net PCINT28: now also U4.13 (B1)
- net OC2A/ renamed PCINT31
- net PCINT31: now also U5.10 (B4)
- net Vsupply renamed +7.5V
- net +7.5V: now also J2.1 (Pin_1), J3.1 (Pin_1), J5.1 (Pin_1), POWER1.1 (Pin_1)
- new net: RP7.2, U5.8 (OE)
- new net: RP5.2, U3.8 (OE)
- new net: J5.3 (Pin_3), R7.1
- new net: J2.3 (Pin_3), R4.1
- new net: J3.3 (Pin_3), R5.1
- new net: J14.2 (Pin_2), RP9.1
- new net: RP6.2, U4.8 (OE)
- new net BT_RST: U4.2 (A1)
- new net P0_0: U3.4 (A3)
- new net P1_6: U4.4 (A3)
- new net P1_7: U4.5 (A4)
- new net P2_0: U4.3 (A2)
- new net P3_6: U3.5 (A4)
- new net RX_3V3: U3.3 (A2)
- new net TX_3V3: U3.2 (A1)
- no-connect marks 6 -> 19
Other:
- note added: "(connect separate\nprocessing module)\n"
- note added: "+5V I2C Pullup\n"
- note added: "Adafruit GPS \nBreakout"
- note added: "CAN SPI Click Breakout"
- note added: "CVT IR Temp"
- note added: "Engine Tach"
- note added: "GB Oil RTD Amp/Breakout"
- note added: "IMU Breakout\n -MPU6050-"
- note added: "LF BHE"
- note added: "Level Shifter\n --GPIO--\n"
- note added: "Level Shifter\n---SPI---\n"
- note added: "Level Shifter\nGPIO+UART"
- note added: "Li-Po Battery\nConnector (2s)\n"
- note added: "RF BHE"
- note added: "RWS BHE\n(output gear)"
- note added: "Real Time Clock\n\n"
- note added: "Ride Height Sensors\n"
- note removed: "I2C Pullup\n"
- note removed: "Level Shifter\n"
- note removed: "Li-Po Battery\nConnector\n"
- note removed: "RTC Module\n"
- moved on the sheet: BT1, C1, C13, C14, C15, C16, C17, C18, C2, C3, C4, C5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

Commit message: added stitching vias
Parts:
- renumbered J1 to ICSP1, U0 to MCU0
Connections:
- net P0_0: now also U3.5 (A4); no longer U3.4 (A3)
- net P2_0: now also U3.4 (A3); no longer U4.3 (A2)
- net P3_6: now also U4.3 (A2); no longer U3.5 (A4)
- net PCINT20: now also U4.13 (B1); no longer U4.12 (B2)
- net PCINT21: now also U4.12 (B2); no longer U4.11 (B3)
- net PCINT22: now also U4.11 (B3); no longer U4.10 (B4)
- net PCINT23: now also U4.10 (B4); no longer J4.5 (Pin_5)
- net PCINT28: now also U5.10 (B4); no longer U4.13 (B1)
- net PCINT31: now also J4.5 (Pin_5); no longer U5.10 (B4)
Changed lines of the file:
@@
 $EndComp
 $Comp
-L Connector_Generic:Conn_02x03_Odd_Even J1
+L Connector_Generic:Conn_02x03_Odd_Even ICSP1
 U 1 1 5D85C07C
 P 10650 1150
-F 0 "J1" H 10700 1467 50  0000 C CNN
+F 0 "ICSP1" H 10700 1467 50  0000 C CNN
 F 1 "ICSP" H 10700 1376 50  0000 C CNN
 F 2 "Connector_PinHeader_2.54mm:PinHeader_2x03_P2.54mm_Vertical" H 10650 1150 50  0001 C CNN
@@
 Crystal Oscillator
 $Comp
-L MCU_Microchip_ATmega:ATmega1284-AU U0
+L MCU_Microchip_ATmega:ATmega1284-AU MCU0
 U 1 1 5D84B034
 P 1550 4350
-F 0 "U0" H 1450 5100 50  0000 C CNN
+F 0 "MCU0" H 1450 5100 50  0000 C CNN
 F 1 "ATmega1284-AU" H 1450 5000 50  0000 C CNN
 F 2 "Package_QFP:TQFP-44_10x10mm_P0.8mm" H 1550 4350 50  0001 C CIN
@@
 CS_3V3
 Text Label 6700 3750 0    50   ~ 0
-PCINT31
+PCINT28
 Text Label 6700 3550 0    50   Italic 0
 SCK
@@
 Text Label 5000 3350 0    50   ~ 0
 TX1
+Text Label 4200 3550 2    50   ~ 0
+P2_0
 Text Label 4200 3750 2    50   ~ 0
-P3_6
-Text Label 4200 3550 2    50   ~ 0
 P0_0
 Text Label 4200 3350 2    50   ~ 0
@@
 SCL
 Text Label 6700 6950 2    39   ~ 0
-PCINT23
+PCINT31
 Wire Notes Line
 	6300 7250 6300 5900
@@
 $EndComp
 Text Label 4200 6050 2    50   ~ 0
-P2_0
+P3_6
 Text Label 4200 6450 2    50   ~ 0
 P1_7
@@
 Text Label 5000 3750 0    50   ~ 0
 PCINT19
+Text Label 5000 5850 0    50   ~ 0
+PCINT20
 Text Label 5000 6050 0    50   ~ 0
-PCINT20
+PCINT21
 Text Label 5000 6250 0    50   ~ 0
-PCINT21
-Text Label 5000 6450 0    50   ~ 0
 PCINT22
 Text Label 2650 7000 2    50   ~ 0
@@
 Text Label 4200 5850 2    50   ~ 0
 BT_RST
-Text Label 5000 5850 0    50   ~ 0
-PCINT28
+Text Label 5000 6450 0    50   ~ 0
+PCINT23
 $Comp
 L power:GND #PWR0165
