File: backdash/rev_1.0/rev_1.0.kicad_pcb (KiCad board)
At the start: 2 copper layers, 114.3 x 67.3 mm, 71 parts, among them J10 RR_rh, J11 Tach, J12 MAX31865, J13 Micro_SD_Card_Det_Hirose_DM3AT, J14 Ulti_GPS_v3, J2 RF_BHE, J3 Output_BHE, J4 IMU_bout, J5 LF_BHE, J6 CVT_IR, J7 LF_rh, J8 LR_rh, J9 RF_rh, SW2 BT_RST, U1 LM1117-5.0, U2 LM1117-3.3, U3 TXB0104D, U4 TXB0104D, U5 TXB0104D, U6 MCP7940N-xSN, U7 RN4871-V/RM118, Y1 16MHz, Y2 32.768 kHz

Commit message: passes DRC, looks pretty
Parts:
- removed J14: Ulti_GPS_v3, baja1920:UltiGPSv3
- added ?: , , F.Cu at (77.0, 178.4)
- added ?: , , F.Cu at (81.6, 60.8)
- added G***: LOGO, baja1920:logo_backdash_front, F.Cu at (104.8, 75.6)
- added G***: LOGO, baja1920:logo_backdash_back, B.Cu at (140.5, 78.0)
- added GPS: Ulti_GPS_v3, baja1920:UltiGPSv3, F.Cu at (164.7, 72.6)
- C17, C18, C4, C5: footprint Capacitor_SMD:C_0201_0603Metric -> Capacitor_SMD:C_0402_1005Metric
- J2: value RF_BHE -> RF
- J3: value Output_BHE -> RWS
- J5: value LF_BHE -> LF
- moved RP9 246.6 mm to (172.3, 80.3)
- moved 5V_PWR 240.7 mm to (90.8, 63.7)
- moved BLE 240.7 mm to (110.9, 45.5)
- moved BT1 240.7 mm to (150.2, 69.1)
- moved BT_PWR 240.7 mm to (119.0, 48.1)
- moved BT_RESET 240.7 mm to (131.5, 45.5)
- moved BT_TX 240.7 mm to (119.0, 43.1)
- moved C1 240.7 mm to (101.0, 68.6)
- moved C10 240.7 mm to (123.1, 52.7)
- moved C11 240.7 mm to (136.7, 58.5)
- moved C12 240.7 mm to (123.1, 58.2)
- moved C13 240.7 mm to (104.4, 85.4)
- moved C14 240.7 mm to (104.4, 81.4)
- moved C15 240.7 mm to (101.7, 85.8)
- moved C16 240.7 mm to (127.3, 70.3)
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- renumbered PLED_3V3 to 3V3_PWR, PLED_5V1 to 5V_PWR, U7 to BLE, D1 to BT_PWR, SW2 to BT_RESET, D2 to BT_TX, CAN1 to CAN, J6 to CVT_IR, ICSP1 to ICSP, J4 to IMU, J7 to LF, J8 to LR, MCU0 to MCU1, POWER1 to POWER, J9 to RF, J10 to RR, J12 to RTD, J11 to TACH, J13 to uSD
Routing:
- net GND: track 178.3 -> 157.5 mm, vias 605 -> 625
- net Net-(J14-Pad2): track 7.25 -> 3.41 mm
- net +5V: track 354.4 -> 350.9 mm
- net /A3: track 22.9 -> 24.0 mm
- net /TX0: track 69.9 -> 70.6 mm
- net /RX0: track 68.3 -> 68.8 mm
Other:
- board text added: "2019-2020 rev 1.0"
- board text added: "Backdash Sensing and Datalogging"
- board text added: "RIDE HEIGHT"
- board text added: "WHEEL SPEED"
